File: Electrical/USB Reset Button/USB Reset Button.sch (KiCad schematic (older format))
At the start: 5 parts

Commit message: Updated Electrical Schematic
Parts:
- removed Q?: 2N3906, Package_TO_SOT_THT:TO-92_Inline, symbol Transistor_BJT:2N3906
- added Q?: Q_PMOS_GSD, symbol Device:Q_PMOS_GSD
- R?: value 1KΩ -> 10KΩ
Changed lines of the file:
@@
 EESchema Schematic File Version 4
+LIBS:USB Reset Button-cache
 EELAYER 26 0
 EELAYER END
@@
 OUTPUT
 NoConn ~ 3800 3550
-Text Label 6300 5850 3    50   ~ 0
-OUTPUT
 $Comp
 L Switch:SW_Push SW?
 U 1 1 5DEC0530
-P 5800 5650
-F 0 "SW?" H 5800 5935 50  0000 C CNN
-F 1 "SW_Push" H 5800 5844 50  0000 C CNN
-F 2 "" H 5800 5850 50  0001 C CNN
-F 3 "" H 5800 5850 50  0001 C CNN
-	1    5800 5650
-	1    0    0    -1
+P 4050 4700
+F 0 "SW?" H 4050 4985 50  0000 C CNN
+F 1 "SW_Push" H 4050 4894 50  0000 C CNN
+F 2 "" H 4050 4900 50  0001 C CNN
+F 3 "" H 4050 4900 50  0001 C CNN
+	1    4050 4700
+	0    -1   -1   0
 $EndComp
 $Comp
 L Device:R R?
 U 1 1 5DEC090B
-P 6000 5800
-F 0 "R?" H 5930 5754 50  0000 R CNN
-F 1 "1KΩ" H 5930 5845 50  0000 R CNN
-F 2 "" V 5930 5800 50  0001 C CNN
-F 3 "~" H 6000 5800 50  0001 C CNN
-	1    6000 5800
+P 4050 5050
+F 0 "R?" H 3980 5004 50  0000 R CNN
+F 1 "10KΩ" H 3980 5095 50  0000 R CNN
+F 2 "" V 3980 5050 50  0001 C CNN
+F 3 "~" H 4050 5050 50  0001 C CNN
+	1    4050 5050
 	-1   0    0    1
-$EndComp
-$Comp
-L Transistor_BJT:2N3906 Q?
-U 1 1 5DEC0B4B
-P 6200 5650
-F 0 "Q?" H 6391 5604 50  0000 L CNN
-F 1 "2N3906" H 6391 5695 50  0000 L CNN
-F 2 "Package_TO_SOT_THT:TO-92_Inline" H 6400 5575 50  0001 L CIN
-F 3 "https://www.fairchildsemi.com/datasheets/2N/2N3906.pdf" H 6200 5650 50  0001 L CNN
-	1    6200 5650
-	1    0    0    1
 $EndComp
 $Comp
 L power:GND #PWR?
 U 1 1 5DEC19A0
-P 6000 5950
-F 0 "#PWR?" H 6000 5700 50  0001 C CNN
-F 1 "GND" V 6005 5822 50  0000 R CNN
-F 2 "" H 6000 5950 50  0001 C CNN
-F 3 "" H 6000 5950 50  0001 C CNN
-	1    6000 5950
+P 4050 5200
+F 0 "#PWR?" H 4050 4950 50  0001 C CNN
+F 1 "GND" V 4055 5072 50  0000 R CNN
+F 2 "" H 4050 5200 50  0001 C CNN
+F 3 "" H 4050 5200 50  0001 C CNN
+	1    4050 5200
 	1    0    0    -1
 $EndComp
-Text Label 6300 5450 1    50   ~ 0
+Text Label 4050 4500 2    50   ~ 0
 INPUT
-Connection ~ 6000 5650
 Wire Wire Line
-	6300 5450 6300 5200
+	4050 4500 4250 4500
 Wire Wire Line
-	6300 5200 5600 5200
+	4450 4800 4450 4900
 Wire Wire Line
-	5600 5200 5600 5650
+	4450 4900 4050 4900
+$Comp
+L Device:Q_PMOS_GSD Q?
+U 1 1 5DF07577
+P 4450 4600
+F 0 "Q?" V 4793 4600 50  0000 C CNN
+F 1 "Q_PMOS_GSD" V 4702 4600 50  0000 C CNN
+F 2 "" H 4650 4700 50  0001 C CNN
+F 3 "~" H 4450 4600 50  0001 C CNN
+	1    4450 4600
+	0    -1   -1   0
+$EndComp
+Connection ~ 4050 4900
+Text Label 4650 4500 0    50   ~ 0
+OUTPUT
 $EndSCHEMATC
